File: electrical/rpu/motion_control/board/board.kicad_sch (KiCad schematic)
At the start: 7 parts, among them J101 HEADER_LEFT, J102 HEADER_BOTTOM, J103 HEADER_RIGHT, U101 ADM7172ACPZ-3.3-R7

Commit message: USB Hub schematic and routing
Parts:
- added D101, D102, D103: PUSB3FR4Z, lcsc_lib:DFN2510-10_L2.5-W1.0-P0.50-BL-2, symbol lcsc_lib:PUSB3FR4Z
- added J104, J105, J106: USB_A, lcsc_lib:USB-A-TH_FUS264-FDSW3K, symbol Connector:USB_A
Connections:
- net GND: now also D101.3 (GND), D101.8 (GND), D102.3 (GND), D102.8 (GND), D103.3 (GND), D103.8 (GND), J104.4 (GND), J104.SH (Shield), J105.4 (GND), J105.SH (Shield), J106.4 (GND), J106.SH (Shield)
- new net: D103.1 (CH1), D103.10 (CH1)
- new net: D103.2 (CH2), D103.9 (CH2)
- new net: D102.1 (CH1), D102.10 (CH1)
- new net: D102.2 (CH2), D102.9 (CH2)
- new net: D101.1 (CH1), D101.10 (CH1)
- new net: D101.2 (CH2), D101.9 (CH2)
- new net USB2Hub/DFP1_D+: D102.5 (CH4), D102.6 (CH4), J105.3 (D+)
- new net USB2Hub/DFP1_D-: D102.4 (CH3), D102.7 (CH3), J105.2 (D-)
- new net USB2Hub/DFP4_D+: D103.5 (CH4), D103.6 (CH4), J106.3 (D+)
- new net USB2Hub/DFP4_D-: D103.4 (CH3), D103.7 (CH3), J106.2 (D-)
- new net USB2Hub/UFP_D+: D101.5 (CH4), D101.6 (CH4), J104.3 (D+)
- new net USB2Hub/UFP_D-: D101.4 (CH3), D101.7 (CH3), J104.2 (D-)
- new net USB2Hub/VBUS: J104.1 (VBUS), J105.1 (VBUS), J106.1 (VBUS)
- no-connect marks 8 -> 14
Other:
- added sheet USB2Hub (USB2Hub.kicad_sch)
- moved on the sheet: C101, C102, C103, J101, J102, J103, U101
