File: electrical/rpu/motion_control/board/cm5-j1.kicad_sch (KiCad schematic)
At the start: 1 part, among them U401 Hirose DF40C-100DS-0.4V

Commit message: USB Hub schematic and routing
Connections:
- no-connect marks 35 -> 36
Changed lines of the file:
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@@
+	)
+	(no_connect
+		(at 36.83 52.07)
 	)
 	(no_connect
