File: electrical/rpu/motion_control/board/board.kicad_pcb (KiCad board)
At the start: 4 copper layers, 106 x 98 mm, 76 parts, among them J101 HEADER_LEFT, J102 HEADER_BOTTOM, J103 HEADER_RIGHT, SW201 TS50810-411-02528, U101 ADM7172ACPZ-3.3-R7, U201 Hirose DF40C-100DS-0.4V, U202 ETH, U203 LSM6DSVTR, U301 Hirose DF40C-100DS-0.4V, U401 Hirose DF40C-100DS-0.4V, U501 TXB0104PW, U502 TXB0104PW, U503 TXB0104PW, U504 TXB0104PW, U601 MCP2518FD-xQBB, U602 MCP2518FD-xQBB, U603 MCP2518FD-xQBB, U604 SN65HVD230, U605 SN65HVD230, U606 SN65HVD230, U607 MCP2518FD-xQBB, U608 MCP2518FD-xQBB, U609 MCP2518FD-xQBB, U610 SN65HVD230, U611 SN65HVD230, U612 SN65HVD230, Y601 40M, Y602 40M, Y603 40M, Y604 40M, Y605 40M, Y606 40M

Commit message: fix some 3d step paths. Fixed warnings
Parts:
- moved C102 1.02 mm to (116.4, 129.9)
- moved R202 1.02 mm to (156.3, 128.6)
- moved SW201 1.02 mm to (156.3, 131.3)
- moved U101 1.02 mm to (119.2, 128.4)
- moved Y603 1.02 mm to (107.0, 93.4)
- moved C607 1.02 mm to (116.4, 48.1)
- moved J102 1.02 mm to (129.1, 132.1)
- moved C602 1.02 mm to (106.2, 60.1)
- moved C201 1.02 mm to (137.0, 86.8)
- moved C202 1.02 mm to (139.0, 86.8)
- moved C203 1.02 mm to (150.1, 45.6)
- moved C204 1.02 mm to (138.8, 59.1)
- moved C205 1.02 mm to (137.1, 59.1)
- moved C501 1.02 mm to (165.6, 109.1)
- moved C502 1.02 mm to (172.8, 108.8)
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Routing:
- net unconnected-(U301-PCIe_nRST-Pad109): track 49.8 -> 0.00 mm, vias 3 -> 0
- net unconnected-(U401-GPIO_3V3_CC_INT0_L-Pad296): track 41.4 -> 0.00 mm, vias 4 -> 0
- net unconnected-(U201-GPIO26-Pad24): track 38.0 -> 0.00 mm, vias 1 -> 0
- net unconnected-(U201-WiFi_nDisable-Pad89): track 20.8 -> 0.00 mm, vias 1 -> 0
- net unconnected-(U201-BT_nDisable-Pad91): track 19.0 -> 0.00 mm, vias 1 -> 0
- net unconnected-(U504-B4-Pad10): track 1.42 -> 0.00 mm, vias 1 -> 0

Commit message: fix hirose 100 pin connector STEP
Other:
- board size 106 x 98 mm -> 106 x 106 mm
Changed lines of the file:
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@@
 		)
 		(property "KiLib_Generator" "package/gullwing"
-			(at 0 0 270)
+			(at 0 0 90)
 			(layer "F.SilkS")
 			(hide yes)
@@
 		)
 		(embedded_fonts no)
-		(model "${KIPRJMOD}/DF40C-100DS.stp"
+		(model "${KIPRJMOD}/lcsc_lib.3dshapes/CONN-SMD_DF40C-100DS-0.4V-51.step"
 			(offset
-				(xyz 33.5 20.385 0)
+				(xyz -0.5 26.525 0)
 			)
 			(scale
@@
 			)
 			(rotate
-				(xyz -90 0 0)
+				(xyz -0 -0 -90)
 			)
 		)
@@
 		)
 		(embedded_fonts no)
-		(model "${KIPRJMOD}/DF40C-100DS.stp"
+		(model "${KIPRJMOD}/lcsc_lib.3dshapes/CONN-SMD_DF40C-100DS-0.4V-51.step"
 			(offset
-				(xyz 33.5 20.385 0)
+				(xyz 33.5 26.5 0)
 			)
 			(scale
@@
 			)
 			(rotate
-				(xyz -90 0 0)
+				(xyz -0 -0 90)
 			)
 		)
@@
 		)
 		(embedded_fonts no)
-		(model "${KIPRJMOD}/DF40C-100DS.stp"
+		(model "${KIPRJMOD}/lcsc_lib.3dshapes/CONN-SMD_DF40C-100DS-0.4V-51.step"
 			(offset
-				(xyz 33.5 20.385 0)
+				(xyz 16.4 48 0)
 			)
 			(scale
@@
 			)
 			(rotate
-				(xyz -90 0 0)
+				(xyz -0 -0 -0)
 			)
 		)
@@
 		(layer "B.SilkS")
 	)
-	(gr_line
-		(start 85 76.999978)
-		(end 85 101.011202)
-		(stroke
-			(width 0.25)
-			(type default)
-		)
-		(layer "Edge.Cuts")
-	)
 	(gr_arc
 		(start 85 76.999978)
@@
 		(end 87.988776 74)
 		(stroke
-			(width 0.25)
-			(type default)
+			(width 0.1)
+			(type solid)
 		)
 		(layer "Edge.Cuts")
 	)
-	(gr_circle
-		(center 88 77)
-		(end 90 77)
+	(gr_line
+		(start 85 134)
+		(end 85 76.999978)
 		(stroke
-			(width 0.25)
+			(width 0.1)
 			(type solid)
 		)
-		(fill no)
 		(layer "Edge.Cuts")
 	)
-	(gr_circle
-		(center 88 101)
-		(end 90 101)
+	(gr_line
+		(start 87.988776 74)
+		(end 90 73.999978)
 		(stroke
-			(width 0.25)
+			(width 0.1)
 			(type solid)
 		)
-		(fill no)
 		(layer "Edge.Cuts")
 	)
-	(gr_arc
-		(start 88 104)
-		(mid 85.882644 103.125277)
-		(end 85 101.011202)
+	(gr_circle
+		(center 88 77)
+		(end 90 77)
 		(stroke
 			(width 0.25)
 			(type default)
 		)
+		(fill no)
 		(layer "Edge.Cuts")
 	)
-	(gr_line
-		(start 90 74)
-		(end 87.988776 74)
+	(gr_circle
+		(center 88 101)
+		(end 90 101)
 		(stroke
 			(width 0.25)
 			(type default)
 		)
+		(fill no)
 		(layer "Edge.Cuts")
 	)
-	(gr_line
-		(start 90 104)
-		(end 88 104)
+	(gr_arc
+		(start 93 40.999998)
+		(mid 94.464467 37.464465)
+		(end 98 36)
 		(stroke
-			(width 0.25)
+			(width 0.1)
 			(type default)
 		)
@@
 	)
 	(gr_arc
-		(start 90 104)
-		(mid 92.12132 104.87868)
-		(end 93 107)
+		(start 93 70.999978)
+		(mid 92.121328 73.121313)
+		(end 90 73.999978)
 		(stroke
-			(width 0.25)
-			(type default)
+			(width 0.1)
+			(type solid)
 		)
 		(layer "Edge.Cuts")
 	)
 	(gr_line
-		(start 93 40.999998)
-		(end 93 70.999978)
-		(stroke
-			(width 0.25)
-			(type default)
-		)
-		(layer "Edge.Cuts")
-	)
-	(gr_arc
-		(start 93 40.999998)
-		(mid 94.464467 37.464465)
-		(end 98 36)
+		(start 93 70.999978)
+		(end 93 40.999998)
 		(stroke
 			(width 0.1)
-			(type default)
+			(type solid)
 		)
 		(layer "Edge.Cuts")
 	)
 	(gr_arc
-		(start 93 70.999978)
-		(mid 92.121328 73.121313)
-		(end 90 73.999978)
+		(start 93 142)
+		(mid 87.343146 139.656854)
+		(end 85 134)
 		(stroke
-			(width 0.25)
-			(type default)
+			(width 0.1)
+			(type solid)
 		)
 		(layer "Edge.Cuts")
 	)
 	(gr_line
-		(start 93 107)
-		(end 93 129.014469)
+		(start 93 142)
+		(end 183 142)
 		(stroke
 			(width 0.1)
-			(type default)
+			(type solid)
 		)
 		(layer "Edge.Cuts")
@@
 		(end 177.999999 36)
 		(stroke
-			(width 0.25)
-			(type default)
+			(width 0.1)
+			(type solid)
 		)
 		(layer "Edge.Cuts")
@@
 	(gr_circle
 		(center 98 49)
-		(end 98 50.6)
+		(end 99.6 49)
 		(stroke
 			(width 0.25)
@@
 	(gr_circle
 		(center 98 129)
-		(end 98 130.6)
+		(end 99.6 129)
 		(stroke
 			(width 0.25)
@@
 		(layer "Edge.Cuts")
 	)
-	(gr_arc
-		(start 98 134)
-		(mid 94.469585 132.540646)
-		(end 93.000021 129.014469)
-		(stroke
-			(width 0.1)
-			(type default)
-		)
-		(layer "Edge.Cuts")
-	)
-	(gr_line
-		(start 98 134)
-		(end 178 134)
+	(gr_circle
+		(center 121.5 65)
+		(end 122.85 65)
 		(stroke
 			(width 0.25)
 			(type default)
 		)
+		(fill no)
 		(layer "Edge.Cuts")
 	)
-	(gr_arc
-		(start 177.999999 36)
-		(mid 181.535534 37.464466)
-		(end 183 41.000001)
+	(gr_circle
+		(center 121.5 113)
+		(end 122.85 113)
 		(stroke
 			(width 0.25)
 			(type default)
 		)
+		(fill no)
 		(layer "Edge.Cuts")
 	)
 	(gr_circle
-		(center 178 49)
-		(end 178 50.6)
+		(center 154.5 65)
+		(end 155.85 65)
 		(stroke
 			(width 0.25)
@@
 	)
 	(gr_circle
-		(center 178 129)
-		(end 178 130.6)
+		(center 154.5 113)
+		(end 155.85 113)
 		(stroke
 			(width 0.25)
@@
 		(layer "Edge.Cuts")
 	)
-	(gr_line
-		(start 183 41.000001)
-		(end 183 71.000018)
+	(gr_arc
+		(start 177.999999 36)
+		(mid 181.535534 37.464466)
+		(end 183 41.000001)
 		(stroke
 			(width 0.1)
-			(type default)
+			(type solid)
 		)
 		(layer "Edge.Cuts")
 	)
-	(gr_arc
-		(start 183 106.999978)
-		(mid 183.882753 104.874614)
-		(end 186.011489 104.000022)
+	(gr_circle
+		(center 178 49)
+		(end 179.6 49)
 		(stroke
-			(width 0.1)
+			(width 0.25)
 			(type default)
 		)
+		(fill no)
 		(layer "Edge.Cuts")
 	)
-	(gr_arc
-		(start 183 128.999978)
-		(mid 181.535542 132.535526)
-		(end 178 134)
+	(gr_circle
+		(center 178 129)
+		(end 179.6 129)
 		(stroke
-			(width 0.1)
+			(width 0.25)
 			(type default)
 		)
+		(fill no)
 		(layer "Edge.Cuts")
 	)
 	(gr_line
-		(start 182.999999 128.999978)
-		(end 183 106.999978)
+		(start 183 41.000001)
+		(end 183 71.000018)
 		(stroke
 			(width 0.1)
-			(type default)
+			(type solid)
 		)
 		(layer "Edge.Cuts")
@@
 		(end 183 71.000018)
 		(stroke
-			(width 0.25)
-			(type default)
+			(width 0.1)
+			(type solid)
 		)
 		(layer "Edge.Cuts")
@@
 		(end 187.99999 74)
 		(stroke
-			(width 0.25)
-			(type default)
-		)
-		(layer "Edge.Cuts")
-	)
-	(gr_line
-		(start 186.011489 104)
-		(end 188 104)
-		(stroke
 			(width 0.1)
-			(type default)
+			(type solid)
 		)
 		(layer "Edge.Cuts")
@@
 		(start 187.99999 74)
 		(mid 190.123771 74.881133)
-		(end 190.999992 77.006946)
+		(end 190.999991 77.006946)
 		(stroke
 			(width 0.1)
-			(type default)
+			(type solid)
 		)
 		(layer "Edge.Cuts")
@@
 		(stroke
 			(width 0.25)
-			(type solid)
+			(type default)
 		)
 		(fill no)
@@
 		(stroke
 			(width 0.25)
-			(type solid)
+			(type default)
 		)
 		(fill no)
 		(layer "Edge.Cuts")
 	)
-	(gr_line
-		(start 190.999991 77.006946)
-		(end 191 101)
+	(gr_arc
+		(start 191 134)
+		(mid 188.656854 139.656854)
+		(end 183 142)
 		(stroke
 			(width 0.1)
-			(type default)
+			(type solid)
 		)
 		(layer "Edge.Cuts")
 	)
-	(gr_arc
-		(start 191 100.999978)
-		(mid 190.121328 103.121313)
-		(end 188 104)
+	(gr_line
+		(start 191 134)
+		(end 190.999991 77.006946)
 		(stroke
 			(width 0.1)
@@
 	)
 	(gr_text "Y"
-		(at 137.975 95.075 180)
+		(at 137.975 95.075 0)
 		(layer "B.SilkS")
 		(effects
@@
 		(polygon
 			(pts
-				(xy 82.875 33.825) (xy 82.875 141.5) (xy 193.325 140.55) (xy 192.8 34.45)
+				(xy 82.875 33.825) (xy 82.875 143.774999) (xy 193.336257 142.824902) (xy 192.8 34.45)
 			)
 		)
@@
 	)
 	(group ""
-		(members "04390424-9219-4608-b293-af997c663d02" "0ee06cab-544e-4df6-955e-ec1705d9cb93"
-			"1b95fe4b-5c5a-4317-b503-a219ef062dd9" "2096aae3-d9d7-4828-8c40-02da9f8e407b"
-			"22aa0548-e07e-4f9e-87f4-214636caf057" "37c695d2-8c5f-4561-8286-6625e50864fe"
-			"39812087-89af-46c3-beee-1c91cd43ac8f" "3b48c0f6-84f5-4b47-a8ab-2adf6fc577db"
-			"48f205ad-165d-4489-86ab-e8750af81029" "62661aa4-386f-4911-b086-3aa5b05199b3"
-			"6b83eb1c-4df5-4f5b-a133-d6e8e231db7a" "6ec02461-4747-4b59-a89b-38fd904688f0"
-			"71e561bd-416d-44a5-87d7-4504e603f78e" "7d6dea04-9053-451b-8654-df2e0c0417b8"
-			"8b1bc49b-91a7-40df-b08b-1502ab33679a" "916c4377-c73d-410f-94b9-03ac4a68e9da"
-			"92359c71-e588-4686-b584-02927276d7de" "ac874e94-7608-41ad-9945-2dfd6583c549"
-			"c1315644-b3fb-4541-a8aa-c13acf9f046f" "cc04929c-8822-497d-8ce7-046f7f1e751e"
-			"cd275ed3-538f-40bd-9069-ffed0535b09b" "d10218f6-167b-4a24-a8fb-f076396e25a7"
-			"d2b7a888-89de-472a-8d41-0d972ad0bb32" "d4686214-46a7-45a1-87d0-d011aa389b7b"
-			"e5cc3970-1f13-422c-921c-13c503c75f0a" "ebe3e71e-25f8-4905-8477-20044af44e98"
-			"f277959d-2127-4af2-8959-deef4cf824a6" "f8b30961-fc6f-4dd2-ad0e-386c4641748f"
+		(members "09e4064a-1915-40fd-ba69-d205a3807c4e" "20257c0d-6f9b-49a0-8c06-f52d86bc611c"
+			"21dbd8d8-4801-4e8d-9db9-a59ab3a00bdf" "27eef713-c82c-452e-a959-b398744b143a"
+			"32f86697-2db5-433a-bfeb-b1fac5db21fe" "3c8a594a-9502-47a5-8146-3074bd2c2572"
+			"4a236ea3-a4cd-4531-9cdd-f9e376ad32b8" "4a448d36-75c0-4672-aff6-af9c02ee0eef"
+			"54511d86-43d3-4981-934f-e81c0ca08014" "5467e89e-322d-4ccb-8566-88a1d0b6c3c7"
+			"71d8e208-01d9-4657-918c-e2a6363665f4" "7aafadea-c0bd-42d4-9cfd-808baed2ae82"
+			"80d00f9e-a660-4955-91c4-5a628cc9f641" "8557b81d-28cd-466c-8fbc-1cf61a236090"
+			"8b6bc2fd-e449-4f0b-b068-bd5c825d04c5" "9b3b7fb8-c3bb-4b8c-8d43-63a20910e7c3"
+			"a82a377d-04fc-451c-a95f-89f8b03e8a4e" "b7d3387d-e144-4277-833f-50b427564885"
+			"bd4732dc-a391-448e-bb4d-6df1e70fc609" "c71449d7-e82b-45c9-9982-c4ede86db5ff"
+			"cab3c44f-f70d-4fe4-8cae-2b88bf87fac5" "cac8b654-9e8f-465c-b7a9-507f56b8ccb2"
+			"e037fe11-6df5-4005-89ce-762967af42cf" "e2c57068-413c-4a89-b21d-535e5aee646f"
+			"f06e0f17-4c2b-4f5b-b0d7-25910784fb18" "f5cb792e-2684-4688-a494-8fea28e304b8"
+			"feb419b6-0c12-4907-b248-b984775a6672"
 		)
 	)

Commit message: USB Hub schematic and routing
Parts:
- added C701: 100n, Capacitor_SMD:C_0402_1005Metric, B.Cu at (150.0, 59.0)
- added C702: 18p, Capacitor_SMD:C_0402_1005Metric, B.Cu at (164.9, 50.4)
- added C703: 18p, Capacitor_SMD:C_0402_1005Metric, B.Cu at (161.1, 50.3)
- added C704: 100n, Capacitor_SMD:C_0402_1005Metric, B.Cu at (153.7, 53.1)
- added C705: 100n, Capacitor_SMD:C_0402_1005Metric, B.Cu at (164.9, 51.4)
- added C706: 100n, Capacitor_SMD:C_0402_1005Metric, B.Cu at (160.8, 60.9)
- added C707: 100n, Capacitor_SMD:C_0402_1005Metric, B.Cu at (162.5, 60.9)
- added C708: 100n, Capacitor_SMD:C_0402_1005Metric, B.Cu at (166.3, 56.4)
- added C709: 100n, Capacitor_SMD:C_0402_1005Metric, B.Cu at (157.2, 51.0)
- added C710: 100n, Capacitor_SMD:C_0402_1005Metric, B.Cu at (164.9, 53.4)
- added C711: 100n, Capacitor_SMD:C_0402_1005Metric, B.Cu at (155.2, 56.9)
- added C712: 100n, Capacitor_SMD:C_0402_1005Metric, B.Cu at (159.7, 60.9)
- added C713: 100n, Capacitor_SMD:C_0402_1005Metric, B.Cu at (158.7, 60.9)
- added D101: PUSB3FR4Z, lcsc_lib:DFN2510-10_L2.5-W1.0-P0.50-BL-2, B.Cu at (149.9, 47.8)
- added D102: PUSB3FR4Z, lcsc_lib:DFN2510-10_L2.5-W1.0-P0.50-BL-2, B.Cu at (98.4, 133.6)
- added D103: PUSB3FR4Z, lcsc_lib:DFN2510-10_L2.5-W1.0-P0.50-BL-2, B.Cu at (174.8, 133.2)
- added J104: USB_A, lcsc_lib:USB-A-TH_FUS264-FDSW3K, F.Cu at (147.0, 47.0)
- added J105: USB_A, lcsc_lib:USB-A-TH_FUS264-FDSW3K, F.Cu at (102.0, 138.0)
- added J106: USB_A, lcsc_lib:USB-A-TH_FUS264-FDSW3K, F.Cu at (174.0, 138.0)
- added R701: 10k, Resistor_SMD:R_0402_1005Metric, B.Cu at (168.7, 54.7)
- added R702: 10k, Resistor_SMD:R_0402_1005Metric, B.Cu at (168.7, 55.7)
- added R703: 10k, Resistor_SMD:R_0402_1005Metric, B.Cu at (168.7, 57.1)
- added R704: 10k, Resistor_SMD:R_0402_1005Metric, B.Cu at (168.7, 58.1)
- added R705: 10k, Resistor_SMD:R_0402_1005Metric, B.Cu at (151.9, 55.4)
- added R706: 100k, Resistor_SMD:R_0402_1005Metric, B.Cu at (155.2, 55.9)
- added R707: 100k, Resistor_SMD:R_0402_1005Metric, B.Cu at (155.2, 54.9)
- added R708: 100k, Resistor_SMD:R_0402_1005Metric, B.Cu at (157.2, 52.0)
- added R709: 100k, Resistor_SMD:R_0402_1005Metric, B.Cu at (155.2, 58.0)
- added R710: 12k, Resistor_SMD:R_0402_1005Metric, B.Cu at (164.9, 52.4)
- added R711: 100k, Resistor_SMD:R_0402_1005Metric, B.Cu at (155.2, 52.6)
- added R712: 100k, Resistor_SMD:R_0402_1005Metric, B.Cu at (155.2, 53.6)
- added TP701: ~{RESET} TP, TestPoint:TestPoint_Keystone_5015_Micro_Mini, B.Cu at (145.3, 56.5)
- added TP702: 3V3 TP, TestPoint:TestPoint_Keystone_5015_Micro_Mini, B.Cu at (141.8, 56.5)
- added TP703: ~{RESET} TP, TestPoint:TestPoint_Keystone_5015_Micro_Mini, B.Cu at (138.3, 56.5)
- added U701: USB2514BT-I/M2, lcsc_lib:QFN-36_L6.0-W6.0-P0.50-BL-EP, B.Cu at (160.5, 56.4)
- added U702: TLV803SDBZR, lcsc_lib:SOT-23-3_L2.9-W1.3-P1.90-LS2.4-BR, B.Cu at (151.5, 57.6)
- added Y701: 24MHz 12pF, Crystal:Crystal_SMD_3225-4Pin_3.2x2.5mm, B.Cu at (162.9, 48.0)
- U601, U602, U603, U607, U608, U609: value MCP2518FD-xQBB -> MCP2518FDT
- moved C203 28.4 mm to (121.7, 45.0)
- moved R201 28.4 mm to (121.7, 51.0)
- moved R202 18.9 mm to (140.7, 139.3), turned to 0 degrees
- moved R301 13.6 mm to (155.8, 132.5), turned to 0 degrees
- moved R302 12.9 mm to (159.9, 132.6)
- moved USB301 12.9 mm to (158.1, 136.9)
- moved SW201 12.8 mm to (146.3, 139.3)
- moved G*** 5.60 mm to (138.0, 72.6)
- moved C204 5.00 mm to (133.8, 59.1)
- moved C205 5.00 mm to (132.1, 59.1)
- moved U202 5.00 mm to (133.0, 47.0)
Routing:
- net /USB2Hub/VBUS: track 0.00 -> 212.0 mm
- net /USB2Hub/DFP1_D+: track 0.00 -> 186.7 mm
- net /USB2Hub/DFP1_D-: track 0.00 -> 186.6 mm
- net /USB2Hub/DFP4_D-: track 0.00 -> 90.8 mm
- net /USB2Hub/DFP4_D+: track 0.00 -> 90.7 mm
- net /U13B/USB2_D+: track 99.0 -> 65.0 mm, vias 0 -> 2
- net /U13B/USB2_D-: track 98.9 -> 65.8 mm, vias 0 -> 2
- net GND: track 221.9 -> 254.1 mm, vias 147 -> 194
- net +3V3: track 41.6 -> 68.6 mm, vias 29 -> 42
- net /USB2Hub/UFP_D+: track 0.00 -> 19.1 mm
- net /USB2Hub/UFP_D-: track 0.00 -> 19.0 mm
- net Net-(U701-RESET_N): track 0.00 -> 15.3 mm
- net +5V: track 98.9 -> 109.6 mm, vias 0 -> 1
- net Net-(U701-XTALIN/CLKIN): track 0.00 -> 7.21 mm
- net Net-(U701-XTALOUT): track 0.00 -> 6.91 mm
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- added copper zone on In1.Cu, net GND

Commit message: fabrication ready
Parts:
- TP703: value ~{RESET} TP -> GND TP
