File: electrical/rpu/motion_control/board/spi-can.kicad_sch (KiCad schematic)
At the start: 36 parts, among them U601 MCP2518FD-xQBB, U602 MCP2518FD-xQBB, U603 MCP2518FD-xQBB, U604 SN65HVD230, U605 SN65HVD230, U606 SN65HVD230, U607 MCP2518FD-xQBB, U608 MCP2518FD-xQBB, U609 MCP2518FD-xQBB, U610 SN65HVD230, U611 SN65HVD230, U612 SN65HVD230, Y601 40M, Y602 40M, Y603 40M, Y604 40M, Y605 40M, Y606 40M

Commit message: USB Hub schematic and routing
Parts:
- removed U601, U602, U603, U607, U608, U609: MCP2518FD-xQBB, Package_SO:SOIC-14_3.9x8.7mm_P1.27mm, symbol Interface_CAN_LIN:MCP2518FD-xQBB
- added U601, U602, U603, U607, U608, U609: MCP2518FDT, Package_SO:SOIC-14_3.9x8.7mm_P1.27mm, symbol lcsc_lib:MCP2518FDT
Connections:
- net +3V3: now also U601.14 (VDD), U602.14 (VDD), U603.14 (VDD), U607.14 (VDD), U608.14 (VDD), U609.14 (VDD)
- net GND: now also U601.15 (VSS), U601.7 (VSS), U602.15 (VSS), U602.7 (VSS), U603.15 (VSS), U603.7 (VSS), U607.15 (VSS), U607.7 (VSS), U608.15 (VSS), U608.7 (VSS), U609.15 (VSS), U609.7 (VSS)
- net SPI00_OSC_1: now also U602.6 (OSC1)
- net SPI00_OSC_2: now also U602.5 (OSC2)
- net SPI01_OSC_1: now also U607.6 (OSC1)
- net SPI01_OSC_2: now also U607.5 (OSC2)
- net SPI0_CLK: now also U602.10 (SCK), U607.10 (SCK)
- net SPI0_CS0: now also U602.13 (~{CS})
- net SPI0_CS1: now also U607.13 (~{CS})
- net SPI0_INT0: now also U602.4 (~{INT})
- net SPI0_INT1: now also U607.4 (~{INT})
- net SPI0_SI: now also U602.11 (SDI), U607.11 (SDI)
- net SPI0_SO: now also U602.12 (SDO), U607.12 (SDO)
- net SPI10_OSC_1: now also U603.6 (OSC1)
- net SPI10_OSC_2: now also U603.5 (OSC2)
- net SPI11_OSC_1: now also U608.6 (OSC1)
- net SPI11_OSC_2: now also U608.5 (OSC2)
- net SPI1_CLK: now also U603.10 (SCK), U608.10 (SCK)
- net SPI1_CS0: now also U603.13 (~{CS})
- net SPI1_CS1: now also U608.13 (~{CS})
- net SPI1_INT0: now also U603.4 (~{INT})
- net SPI1_INT1: now also U608.4 (~{INT})
- net SPI1_SI: now also U603.11 (SDI), U608.11 (SDI)
- net SPI1_SO: now also U603.12 (SDO), U608.12 (SDO)
- net SPI40_OSC_1: now also U601.6 (OSC1)
- net SPI40_OSC_2: now also U601.5 (OSC2)
- net SPI41_OSC_1: now also U609.6 (OSC1)
- net SPI41_OSC_2: now also U609.5 (OSC2)
- net SPI4_CLK: now also U601.10 (SCK), U609.10 (SCK)
- net SPI4_CS0: now also U601.13 (~{CS})
- net SPI4_CS1: now also U609.13 (~{CS})
- net SPI4_INT0: now also U601.4 (~{INT})
- net SPI4_INT1: now also U609.4 (~{INT})
- net SPI4_SI: now also U601.11 (SDI), U609.11 (SDI)
- net SPI4_SO: now also U601.12 (SDO), U609.12 (SDO)
- net at U605.1 (D): now also U602.1 (TXCAN)
- net at U605.4 (R): now also U602.2 (RXCAN)
- net at U612.1 (D): now also U609.1 (TXCAN)
- net at U612.4 (R): now also U609.2 (RXCAN)
- net at U604.1 (D): now also U601.1 (TXCAN)
- net at U604.4 (R): now also U601.2 (RXCAN)
- net at U611.1 (D): now also U608.1 (TXCAN)
- net at U611.4 (R): now also U608.2 (RXCAN)
- net at U606.1 (D): now also U603.1 (TXCAN)
- net at U606.4 (R): now also U603.2 (RXCAN)
- net at U610.1 (D): now also U607.1 (TXCAN)
- net at U610.4 (R): now also U607.2 (RXCAN)

Commit message: fabrication ready
Parts:
- Y601, Y602, Y603, Y604, Y605, Y606: LCSC C5444549 -> C7473041
Changed lines of the file:
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@@
 			)
 		)
-		(property "LCSC" "C5444549"
+		(property "LCSC" "C7473041"
 			(at 36.83 139.7 0)
 			(hide yes)
@@
 			)
 		)
-		(property "LCSC" "C5444549"
+		(property "LCSC" "C7473041"
 			(at 177.8 139.7 0)
 			(hide yes)
@@
 			)
 		)
-		(property "LCSC" "C5444549"
+		(property "LCSC" "C7473041"
 			(at 176.53 91.44 0)
 			(hide yes)
@@
 			)
 		)
-		(property "LCSC" "C5444549"
+		(property "LCSC" "C7473041"
 			(at 175.26 44.45 0)
 			(hide yes)
@@
 			)
 		)
-		(property "LCSC" "C5444549"
+		(property "LCSC" "C7473041"
 			(at 36.83 91.44 0)
 			(hide yes)
@@
 			)
 		)
-		(property "LCSC" "C5444549"
+		(property "LCSC" "C7473041"
 			(at 36.83 44.45 0)
 			(hide yes)
