Commit message: fix(sim-model): update link mass and add neck joints

File: sim-model/urdf/asimov_1.urdf (robot description, URDF)
Before this commit: robot asimov_1, 26 links, 25 joints
Links:
- link left_ankle_pitch_link: mass 0.2730901194 -> 0.3030901194
- link left_ankle_roll_link: mass 0.44468 -> 0.48968
- link left_elbow_link: mass 0.6623176013 -> 0.6973176013
- link left_hip_pitch_link: mass 1.056301122 -> 1.101301122
- link left_hip_roll_link: mass 0.4143681394 -> 0.4493681394
- link left_hip_yaw_link: mass 1.866570164 -> 1.921570164
- link left_knee_link: mass 2.391141511 -> 2.466141511
- link left_shoulder_pitch_link: mass 0.5991571366 -> 0.6241571366
- link left_shoulder_roll_link: mass 1.31322813 -> 1.36322813
- link left_shoulder_yaw_link: mass 0.7122617553 -> 0.7372617553
- link left_wrist_yaw_link: mass 0.05805879065 -> 0.06805879065
- link neck_pitch_link: mass 0.3940556092 -> 0.4140556092
- link neck_yaw_link: mass 0.5327893053 -> 0.5527893053
- link pelvis_link: mass 3.506912512 -> 3.606912512
- link right_ankle_pitch_link: mass 0.2730891716 -> 0.3030891716
- link right_ankle_roll_link: mass 0.44468 -> 0.48968
- link right_elbow_link: mass 0.6623142589 -> 0.6973142589
- link right_hip_pitch_link: mass 1.056297429 -> 1.101297429
- link right_hip_roll_link: mass 0.4148250006 -> 0.4498250006
- link right_hip_yaw_link: mass 1.866472204 -> 1.921472204
- link right_knee_link: mass 2.391101676 -> 2.466101676
- link right_shoulder_pitch_link: mass 0.5991561057 -> 0.6241561057
- link right_shoulder_roll_link: mass 1.313222376 -> 1.363222376
- link right_shoulder_yaw_link: mass 0.7122617553 -> 0.7372617553
- link right_wrist_yaw_link: mass 0.05805951068 -> 0.06805951068
- link waist_yaw_link: mass 8.208501581 -> 10.508501581
Joints:
- removed joint neck_pitch_link_fixed
- removed joint neck_yaw_link_fixed
- added joint neck_pitch_joint: type revolute, parent neck_yaw_link, child neck_pitch_link, origin xyz=0 0 0.03735 rpy=0 0 0, axis 0 1 0, limit lower=-0.258 upper=0.527 effort=12 velocity=9.32
- added joint neck_yaw_joint: type revolute, parent waist_yaw_link, child neck_yaw_link, origin xyz=-0.01659877455 0 0.3781670296 rpy=0 0 0, axis 0 0 1, limit lower=-1.57 upper=1.57 effort=12 velocity=9.32
